File: S3_module/S3_module.kicad_sch (KiCad schematic)
At the start: 24 parts

Commit message: add power
Parts:
- added C? (x8): (no value), symbol Device:C_Small
- added D?: (no value), symbol Device:LED
- added J?: (no value), symbol Connector:USB_C_Receptacle_USB2.0
- added R? (x7): (no value), symbol Device:R_Small
- added SW? (x2): (no value), symbol Switch:SW_Push
- added U?: (no value), symbol Regulator_Linear:LD1117S33TR_SOT223
- C?: value (none) -> 100n
- C?: value (none) -> 10n
- R?: value (none) -> 10k
- SW?: value (none) -> SW_DIP_x01
- U?: value ESP32-S3-WROOM-1 -> (none); footprint Espressif:ESP32-S3-WROOM-1 -> (none)
- U?: value (none) -> SN74LVC1G17DCKR; footprint (none) -> Package_TO_SOT_SMD:SOT-353_SC-70-5_Handsoldering
Connections:
- net DC is gone; now on net CS: J?.6 (Pin_6)
- net GND: now also U?.1 (GND), U?.40 (GND), U?.41 (GND), C?.1, C?.2, C?.2, C?.2, C?.2, C?.2, C?.2, C?.2, D?.1 (K), J?.A1 (GND), J?.A12 (GND), J?.B1 (GND), J?.B12 (GND), J?.S1 (SHIELD), R?.2, R?.2, SW?.1, SW?.1, U?.1 (GND)
- net RES: now also U?.27 (GPIO0/BOOT), SW?.2
- net SCL: now also U?.20 (GPIO12/TOUCH11/ADC2_CH0/FSPICS0/FSPIIO4/SUBSPICS0)
- net SDA: now also U?.19 (GPIO11/TOUCH11/ADC2_CH0/FSPICS0/FSPIIO4/SUBSPICS0)
- net VCC: now also U?.2 (3V3), C?.1, C?.1, C?.1, R?.1, R?.1, U?.2 (VO)
- net at U?.13 (GPIO19/U1RTS/ADC2_CH8/CLK_OUT2/USB_D-): now also R?.2
- net at U?.14 (GPIO20/U1CTS/ADC2_CH9/CLK_OUT1/USB_D+): now also R?.2
- net EN: now reaches U?.3 (EN)
- net EN: now also C?.1, R?.2, R?.2
- new net: D?.2 (A), R?.2
- new net: C?.2, R?.1, SW?.2
- new net +5V: C?.1, J?.A4 (VBUS), J?.A9 (VBUS), J?.B4 (VBUS), J?.B9 (VBUS), U?.3 (VI)
- new net CC1: J?.A5 (CC1), R?.1
- new net CC2: J?.B5 (CC2), R?.1
- new net D+: C?.1, J?.A6 (D+), J?.B6 (D+), R?.1
- new net D-: C?.1, J?.A7 (D-), J?.B7 (D-), R?.1
- no-connect marks 0 -> 6
Other:
- note added: "DISPLAY"
- note added: "ROTARY ENCODER"
- note added: "USB C AND LDO"
- moved on the sheet: J?, SW?, U?

Commit message: add footprint
Parts:
- removed SW? (x6): SW_DIP_x01, symbol Switch:SW_DIP_x01
- removed SW? (x2): (no value), symbol Switch:SW_Push
- added C10, C5, C7, C9: C_Small, Capacitor_SMD:C_0805_2012Metric_Pad1.18x1.45mm_HandSolder, symbol Device:C_Small
- added D1, D2, D4, D5: WS2812B, LED_SMD:LED_WS2812B_PLCC4_5.0x5.0mm_P3.2mm, symbol LED:WS2812B
- added D10, D11, D6, D7, D8, D9: 1N4148WS, Diode_SMD:D_SOD-323, symbol Diode:1N4148WS
- added J2: Conn_01x05_Male, Connector_PinHeader_2.54mm:PinHeader_1x05_P2.54mm_Vertical, symbol Connector:Conn_01x05_Male
- added SW1, SW2: SW_4, Kayasu:SW_3x4x2.5mm, symbol Kayasu:SW_4
- added SW4, SW5, SW6, SW7, SW8, SW9: SW_Push, Button_Switch_Keyboard:SW_Cherry_MX_1.00u_Plate, symbol Switch:SW_Push
- C1, C11, C12, C2, C3, C4, C6, C8: renamed from C?; value (none) -> C_Small; footprint (none) -> Capacitor_SMD:C_0805_2012Metric_Pad1.18x1.45mm_HandSolder
- C13, C14, C15: renamed from C?; value 10n -> C_Small; footprint (none) -> Capacitor_SMD:C_0805_2012Metric_Pad1.18x1.45mm_HandSolder
- C16, C17, C18: renamed from C?; value 100n -> C_Small; footprint (none) -> Capacitor_SMD:C_0805_2012Metric_Pad1.18x1.45mm_HandSolder
- D3: renamed from D?; value (none) -> LED; footprint (none) -> LED_SMD:LED_0805_2012Metric_Pad1.15x1.40mm_HandSolder
- J1: renamed from J?; value (none) -> USB_C_Receptacle_USB2.0; footprint (none) -> Connector_USB:USB_C_Receptacle_HRO_TYPE-C-31-M-12
- J3: renamed from J?; value DISPLAY -> Conn_01x08_Female; footprint (none) -> Connector_PinHeader_2.54mm:PinHeader_1x08_P2.54mm_Vertical
- R1, R2, R3, R4, R5, R6, R7: renamed from R?; value (none) -> R_Small; footprint (none) -> Resistor_SMD:R_0805_2012Metric_Pad1.20x1.40mm_HandSolder
- R10, R11, R12, R13, R8, R9: renamed from R?; value 10k -> R_Small; footprint (none) -> Resistor_SMD:R_0805_2012Metric_Pad1.20x1.40mm_HandSolder
- SW3: renamed from SW?; footprint (none) -> Rotary_Encoder:RotaryEncoder_Alps_EC11E-Switch_Vertical_H20mm
- U1: renamed from U?; value (none) -> LD1117S33TR_SOT223; footprint (none) -> Package_TO_SOT_SMD:SOT-223-3_TabPin2
- U2: renamed from U?; value (none) -> ESP32-S3-WROOM-1; footprint (none) -> Espressif:ESP32-S3-WROOM-1
- U3, U4, U5: renamed from U?; value SN74LVC1G17DCKR -> 74LVC1G17
Connections:
- net +5V: now also C10.2, C5.2, C7.2, C9.2, D1.1 (VDD), D2.1 (VDD), D4.1 (VDD), D5.1 (VDD)
- net CS: now also U2.7 (GPIO7/TOUCH7/ADC1_CH6); no longer J3.6 (Pin_6)
- net GND: now also C10.1, C5.1, C7.1, C9.1, D1.3 (VSS), D2.3 (VSS), D4.3 (VSS), D5.3 (VSS), SW1.1, SW2.1
- net RES: now also SW1.2
- net at C3.2, R2.1: now also SW2.2
- net IO8: now reaches U2.12 (GPIO8/TOUCH8/ADC1_CH7/SUBSPICS1)
- net IO3: now reaches U2.15 (GPIO3/TOUCH3/ADC1_CH2)
- net IO3: now also J2.3 (Pin_3)
- net SW_1: now reaches U2.16 (GPIO46)
- net SW_1: now also SW4.1, SW5.1
- net IO9: now reaches U2.17 (GPIO9/TOUCH9/ADC1_CH8/FSPIHD/SUBSPIHD)
- net IO10: now reaches U2.18 (GPIO10/TOUCH10/ADC1_CH9/FSPICS0/FSPIIO4/SUBSPICS0)
- net SW_A: now reaches U2.23 (GPIO21)
- net SW_A: now also D10.1 (K), D6.1 (K), D8.1 (K)
- net SW_3: now reaches U2.24 (GPIO47/SPICLK_P/SUBSPICLK_P_DIFF)
- net SW_3: now also SW8.1, SW9.1
- net SW_2: now reaches U2.25 (GPIO48/SPICLK_N/SUBSPICLK_N_DIFF)
- net SW_2: now also SW6.1, SW7.1
- net SW_B: now reaches U2.26 (GPIO45)
- net SW_B: now also D11.1 (K), D7.1 (K), D9.1 (K)
- net IO2: now reaches U2.38 (GPIO2/TOUCH2/ADC1_CH1)
- net IO2: now also J2.4 (Pin_4)
- net IO1: now reaches U2.39 (GPIO1/TOUCH1/ADC1_CH0)
- net IO1: now also J2.5 (Pin_5)
- net IO4: now reaches U2.4 (GPIO4/TOUCH4/ADC1_CH3)
- net IO4: now also J2.2 (Pin_2)
- net IO5: now reaches U2.5 (GPIO5/TOUCH5/ADC1_CH4)
- net IO5: now also J2.1 (Pin_1)
- net DC: now reaches U2.6 (GPIO6/TOUCH6/ADC1_CH5)
- net DC: now also J3.6 (Pin_6)
- new net: D11.2 (A), SW9.2
- new net: D1.2 (DOUT), D2.4 (DIN)
- new net: D7.2 (A), SW5.2
- new net: D6.2 (A), SW4.2
- new net: D10.2 (A), SW8.2
- new net: D2.2 (DOUT), D4.4 (DIN)
- new net: D8.2 (A), SW6.2
- new net: D9.2 (A), SW7.2
- new net: D4.2 (DOUT), D5.4 (DIN)
- new net DIN: D1.4 (DIN)
Other:
- note added: "HEADER"
- note added: "SWITCH MATRIX"
- note added: "WS2812"
- moved on the sheet: C11, C12, R6, R7

Commit message: layout
Parts:
- removed J3: Conn_01x08_Female, Connector_PinHeader_2.54mm:PinHeader_1x08_P2.54mm_Vertical, symbol Connector:Conn_01x08_Female
- added U6: 0.96_80x160_IPS, Kayasu:0.96_80x160_IPS, symbol Kayasu:0.96_80x160_IPS
- C1, C6: value C_Small -> 1u
- C10, C3, C4, C5, C7, C9: value C_Small -> 0.1u
- C11, C12: value C_Small -> NC
- C13, C14, C15: value C_Small -> 10n
- C16, C17, C18: value C_Small -> 100n
- C2: value C_Small -> 22u
- C8: value C_Small -> 4.7u
- R1, R10, R11, R12, R13, R5, R8, R9: value R_Small -> 10k
- R2, R6, R7: value R_Small -> 0
- R3, R4: value R_Small -> 5.1k
- SW1, SW2: value SW_4 -> (none); footprint Kayasu:SW_3x4x2.5mm -> (none)
- SW4, SW5, SW6, SW7, SW8, SW9: footprint Button_Switch_Keyboard:SW_Cherry_MX_1.00u_Plate -> Switch_Keyboard_Cherry_MX:SW_Cherry_MX_Plate_1.00u
Connections:
- net GND: now also U6.1 (GND)
- net R_A: now also U2.21 (GPIO13/TOUCH13/ADC2_CH2/FSPIQ/FSPIIO7/SUBSPIQ)
- net R_B: now also U2.22 (GPIO14/TOUCH14/ADC2_CH3/FSPIWP/FSPIDQS/SUBSPIWP)
- net R_Z: now also U2.8 (GPIO15/U0RTS/ADC2_CH4/XTAL_32K_P)
- net VCC: now also U6.2 (VCC)
- net USB_D+: now reaches R6.2, U2.14 (GPIO20/U1CTS/ADC2_CH9/CLK_OUT1/USB_D+)
- net USB_D-: now reaches R7.2, U2.13 (GPIO19/U1RTS/ADC2_CH8/CLK_OUT2/USB_D-)
- net CS renamed IO7
- net IO7: now also U6.7 (CS)
- net DC renamed IO6
- net IO6: now also U6.6 (DC)
- net RES renamed BOOT
- net BOOT: now also U6.5 (RES)
- net SCL renamed DIS_CLK
- net DIS_CLK: now also U6.3 (SCL)
- net SDA renamed DIS_SDA
- net DIS_SDA: now also U6.4 (SDA)
- no-connect marks 6 -> 17
Other:
- note added: "CANT BE USED"
