File: S3_module/S3_module.kicad_pcb (KiCad board)
At the start: 2 copper layers, 59 parts, among them J1 USB_C_Receptacle_USB2.0, J2 Conn_01x05_Male, J3 Conn_01x08_Female, SW1 SW_4, SW2 SW_4, SW3 RotaryEncoder_Switch, SW4 SW_Push, SW5 SW_Push, SW6 SW_Push, SW7 SW_Push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

Commit message: layout
Parts:
- removed J3: Conn_01x08_Female, Connector_PinHeader_2.54mm:PinHeader_1x08_P2.54mm_Vertical
- added U6: 0.96_80x160_IPS, Kayasu:0.96_80x160_IPS, F.Cu at (139.3, 86.0)
- C1, C6: value C_Small -> 1u
- C10, C3, C4, C5, C7, C9: value C_Small -> 0.1u
- C11, C12: value C_Small -> NC
- C13, C14, C15: value C_Small -> 10n
- C16, C17, C18: value C_Small -> 100n
- C2: value C_Small -> 22u
- C8: value C_Small -> 4.7u
- R1, R10, R11, R12, R13, R5, R8, R9: value R_Small -> 10k
- R2, R6, R7: value R_Small -> 0
- R3, R4: value R_Small -> 5.1k
- SW4, SW5, SW6, SW7, SW8, SW9: footprint Button_Switch_Keyboard:SW_Cherry_MX_1.00u_Plate -> Switch_Keyboard_Cherry_MX:SW_Cherry_MX_Plate_1.00u
- moved J1 87.2 mm to (177.8, 125.1), turned to 90 degrees
- moved C18 84.0 mm to (101.6, 93.3)
- moved C7 82.6 mm to (99.1, 110.1), turned to -90 degrees
- moved R13 78.7 mm to (106.7, 92.1)
- moved C13 78.2 mm to (95.5, 90.8)
- moved D11 76.3 mm to (160.0, 136.5)
- moved U2 75.3 mm to (168.9, 94.0)
- moved C5 72.1 mm to (101.6, 110.1), turned to -90 degrees
- moved C16 68.3 mm to (100.3, 88.3)
- moved R12 63.1 mm to (110.5, 92.1)
- moved C17 62.9 mm to (100.3, 90.8)
- moved R9 62.3 mm to (110.5, 88.3)
- moved C14 61.8 mm to (95.5, 93.3)
- moved J2 60.7 mm to (166.4, 145.4), turned to 90 degrees
- moved D5 59.3 mm to (100.3, 136.5)
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Connections:
- net Net-(R6-Pad2) renamed /USB_D+
- net Net-(R7-Pad2) renamed /USB_D-
- net RES renamed /BOOT
- U2 pad 19: SDA -> /DIS_SDA
- U2 pad 20: SCL -> /DIS_CLK
- U2 pad 21: unconnected-(U2-Pad21) -> R_A
- U2 pad 22: unconnected-(U2-Pad22) -> R_B
- U2 pad 6: DC -> /IO6
- U2 pad 7: CS -> /IO7
- U2 pad 8: unconnected-(U2-Pad8) -> R_Z
Routing:
- net /D-: track 0.00 -> 29.7 mm
- net /D+: track 0.00 -> 28.3 mm
- net VCC: track 0.00 -> 14.8 mm, vias 0 -> 5
- net /+5V: track 0.00 -> 12.5 mm
- net GND: track 0.00 -> 10.2 mm, vias 0 -> 5
- net /USB_D-: track 0.00 -> 8.76 mm
- net /USB_D+: track 0.00 -> 7.44 mm
- added copper zone on In2.Cu, net GND
- added copper zone on In1.Cu, net VCC
Other:
- board outline added: 86.9 x 63.9 mm
- copper layers 2 -> 4

Commit message: restore backup
Parts:
- moved C14 26.2 mm to (121.1, 88.1)
- moved C5 24.7 mm to (94.7, 133.8)
- moved SW1 21.7 mm to (170.2, 107.7), turned to 90 degrees
- moved C17 21.4 mm to (121.1, 85.9)
- moved SW5 19.1 mm to (152.4, 138.4)
- moved SW8 19.1 mm to (152.4, 119.4)
- moved C10 17.8 mm to (94.7, 127.5)
- moved C13 17.7 mm to (113.0, 88.1)
- moved U3 14.0 mm to (108.2, 89.4), turned to 90 degrees
- moved C16 12.9 mm to (113.0, 85.9)
- moved R2 12.6 mm to (156.7, 93.0)
- moved D3 12.1 mm to (167.1, 115.6), turned to 90 degrees
- moved C15 11.6 mm to (103.9, 88.1)
- moved C9 11.5 mm to (94.7, 121.2)
- moved C12 10.9 mm to (156.7, 97.5), turned to 180 degrees
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Routing:
- net GND: track 10.2 -> 104.8 mm, vias 5 -> 44
- net /+5V: track 12.5 -> 57.9 mm
- net VCC: track 14.8 -> 38.9 mm, vias 5 -> 16
- net /Rotary_A: track 0.00 -> 17.3 mm
- net Net-(D10-Pad2): track 0.00 -> 15.4 mm
- net /BOOT: track 0.00 -> 13.9 mm
- net Net-(D8-Pad2): track 0.00 -> 11.9 mm
- net Net-(D6-Pad2): track 0.00 -> 11.6 mm
- net Net-(C13-Pad1): track 0.00 -> 11.1 mm
- net Net-(C14-Pad1): track 0.00 -> 10.0 mm
- net Net-(C15-Pad1): track 0.00 -> 9.17 mm
- net /Rotary_Z: track 0.00 -> 8.93 mm
- net /EN: track 0.00 -> 8.31 mm
- net /Rotary_B: track 0.00 -> 8.28 mm
- net Net-(C3-Pad2): track 0.00 -> 7.11 mm
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Other:
- board size 86.9 x 63.9 mm -> 90.9 x 63.9 mm

Commit message: route, to be revise
Parts:
- moved SW5 38.1 mm to (114.3, 138.4)
- moved SW9 38.1 mm to (152.4, 138.4)
- moved R1 12.8 mm to (156.7, 97.5)
- moved C12 11.2 mm to (159.3, 108.5), turned to 0 degrees
- moved R7 2.70 mm to (155.4, 105.4)
- moved R6 2.54 mm to (157.5, 105.4)
- moved C11 1.98 mm to (155.4, 101.3), turned to 90 degrees
- moved D11 1.78 mm to (162.1, 141.5)
- moved D7 1.78 mm to (123.4, 141.5)
- moved D9 1.78 mm to (143.0, 141.5)
- moved D3 0.25 mm to (167.4, 115.6)
Routing:
- net SW_2: track 0.00 -> 95.7 mm, vias 0 -> 3
- net SW_B: track 0.00 -> 92.7 mm, vias 0 -> 2
- net R_Z: track 0.00 -> 88.1 mm, vias 0 -> 2
- net SW_A: track 0.00 -> 87.1 mm, vias 0 -> 2
- net /IO5: track 0.00 -> 85.2 mm, vias 0 -> 3
- net SW_1: track 0.00 -> 80.3 mm, vias 0 -> 2
- net /+5V: track 57.9 -> 138.0 mm, vias 0 -> 2
- net /IO4: track 0.00 -> 76.6 mm, vias 0 -> 3
- net R_A: track 0.00 -> 68.1 mm, vias 0 -> 3
- net /IO1: track 0.00 -> 64.1 mm
- net SW_3: track 0.00 -> 63.3 mm, vias 0 -> 3
- net R_B: track 0.00 -> 63.1 mm, vias 0 -> 4
- net /IO2: track 0.00 -> 62.7 mm
- net /IO3: track 0.00 -> 59.4 mm, vias 0 -> 4
- net /BOOT: track 13.9 -> 66.5 mm, vias 0 -> 2
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Other:
- board size 90.9 x 63.9 mm -> 93.2 x 63.9 mm

Commit message: V1
Routing:
- net R_B: track 63.1 -> 67.5 mm
- net /IO7: track 24.7 -> 28.4 mm
- net /IO5: track 85.2 -> 82.3 mm
- net Net-(D3-Pad2): track 0.04 -> 2.33 mm
- net Net-(C3-Pad2): track 42.5 -> 43.9 mm
- net /+5V: track 138.0 -> 136.6 mm
- net /IO4: track 76.6 -> 77.6 mm
- net GND: track 103.2 -> 102.4 mm, vias 45 -> 44
- net /DIS_CLK: track 42.6 -> 43.5 mm
- net R_Z: track 88.1 -> 88.9 mm
- net R_A: track 68.1 -> 68.0 mm, vias 3 -> 2
Other:
- board text added: "0.1u"
- board text added: "10k"
- board text added: "10n"

Commit message: last version
Routing:
- net /D-: track 38.7 -> 37.1 mm
- net /IO1: track 64.1 -> 62.8 mm, vias 0 -> 1
- net SW_B: track 92.7 -> 93.3 mm
Other:
- board size 93.2 x 63.9 mm -> 91.8 x 63.9 mm
- board text added: "IO5 IO4 IO3 IO2 IO1"
- board text added: "Li HK 2022-05-01"
Changed lines of the file:
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@@
   (gr_line (start 179.451 84.709) (end 179.197 84.963) (layer "F.SilkS") (width 0.15))
   (gr_line (start 179.197 84.963) (end 181.356 84.963) (layer "F.SilkS") (width 0.15))
-  (gr_rect (start 183.134 84.074) (end 89.916 147.955) (layer "Edge.Cuts") (width 0.1) (fill none))
+  (gr_rect (start 181.737 84.074) (end 89.916 147.955) (layer "Edge.Cuts") (width 0.1) (fill none))
   (gr_text "10n" (at 99.218762 88.011) (layer "F.SilkS")
     (effects (font (size 1 1) (thickness 0.15)))
+  )
+  (gr_text "Li HK\n2022-05-01" (at 170.942 137.033) (layer "F.SilkS")
+    (effects (font (size 1 1) (thickness 0.15)))
+  )
+  (gr_text "IO5 IO4 IO3 IO2 IO1" (at 171.577 143.129) (layer "F.SilkS")
+    (effects (font (size 0.8 0.8) (thickness 0.15)))
   )
   (gr_text "10k" (at 99.266381 90.072629) (layer "F.SilkS")
@@
   (via (at 108.966 123.698) (size 0.8) (drill 0.4) (layers "F.Cu" "B.Cu") (net 5))
   (segment (start 108.966 123.698) (end 115.316 123.698) (width 0.5) (layer "B.Cu") (net 5))
-  (segment (start 155.448 102.3835) (end 154.4105 102.3835) (width 0.2) (layer "F.Cu") (net 6))
   (segment (start 168.069739 124.646102) (end 172.828889 124.646102) (width 0.2) (layer "F.Cu") (net 6))
-  (segment (start 153.416 103.378) (end 153.416 105.156) (width 0.2) (layer "F.Cu") (net 6))
   (segment (start 172.828889 124.696111) (end 173.606111 124.696111) (width 0.2) (layer "F.Cu") (net 6))
   (segment (start 173.606111 124.696111) (end 173.755 124.845) (width 0.2) (layer "F.Cu") (net 6))
-  (segment (start 153.416 105.156) (end 154.67 106.41) (width 0.2) (layer "F.Cu") (net 6))
-  (segment (start 154.4105 102.3835) (end 153.416 103.378) (width 0.2) (layer "F.Cu") (net 6))
   (segment (start 156.3132 107.2752) (end 156.3132 112.889563) (width 0.2) (layer "F.Cu") (net 6))
+  (segment (start 154.051 105.013) (end 155.448 106.41) (width 0.2) (layer "F.Cu") (net 6))
   (segment (start 172.72 125.102778) (end 172.828889 124.993889) (width 0.2) (layer "F.Cu") (net 6))
   (segment (start 172.828889 124.993889) (end 173.755 124.993889) (width 0.2) (layer "F.Cu") (net 6))
   (segment (start 155.448 106.41) (end 156.3132 107.2752) (width 0.2) (layer "F.Cu") (net 6))
   (segment (start 173.089 125.845) (end 172.72 125.476) (width 0.2) (layer "F.Cu") (net 6))
-  (segment (start 154.67 106.41) (end 155.448 106.41) (width 0.2) (layer "F.Cu") (net 6))
+  (segment (start 154.051 103.7805) (end 154.051 105.013) (width 0.2) (layer "F.Cu") (net 6))
   (segment (start 156.3132 112.889563) (end 168.069739 124.646102) (width 0.2) (layer "F.Cu") (net 6))
+  (segment (start 155.448 102.3835) (end 154.051 103.7805) (width 0.2) (layer "F.Cu") (net 6))
   (segment (start 173.755 125.845) (end 173.089 125.845) (width 0.2) (layer "F.Cu") (net 6))
   (segment (start 172.828889 124.646102) (end 172.828889 124.696111) (width 0.2) (layer "F.Cu") (net 6))
@@
   (segment (start 120.65 114.3) (end 123.698 117.348) (width 0.3) (layer "F.Cu") (net 18))
   (segment (start 116.84 114.3) (end 120.65 114.3) (width 0.3) (layer "F.Cu") (net 18))
-  (segment (start 163.379113 142.528) (end 161.832 142.528) (width 0.3) (layer "F.Cu") (net 19))
-  (segment (start 179.07 117.856) (end 176.87552 120.05048) (width 0.3) (layer "F.Cu") (net 19))
-  (segment (start 176.87552 120.05048) (end 176.87552 129.031593) (width 0.3) (layer "F.Cu") (net 19))
-  (segment (start 178.054 108.204) (end 179.07 109.22) (width 0.3) (layer "F.Cu") (net 19))
+  (segment (start 164.558 142.528) (end 161.832 142.528) (width 0.3) (layer "F.Cu") (net 19))
+  (segment (start 178.943 117.983) (end 176.276 120.65) (width 0.3) (layer "F.Cu") (net 19))
+  (segment (start 176.276 120.65) (end 176.276 130.81) (width 0.3) (layer "F.Cu") (net 19))
+  (segment (start 176.276 130.81) (end 164.558 142.528) (width 0.3) (layer "F.Cu") (net 19))
   (segment (start 175.895 102.235) (end 175.895 103.48) (width 0.3) (layer "F.Cu") (net 19))
-  (segment (start 176.87552 129.031593) (end 163.379113 142.528) (width 0.3) (layer "F.Cu") (net 19))
+  (segment (start 178.054 108.204) (end 178.943 109.093) (width 0.3) (layer "F.Cu") (net 19))
   (segment (start 175.768 102.108) (end 175.895 102.235) (width 0.3) (layer "F.Cu") (net 19))
-  (segment (start 179.07 109.22) (end 179.07 117.856) (width 0.3) (layer "F.Cu") (net 19))
+  (segment (start 178.943 109.093) (end 178.943 117.983) (width 0.3) (layer "F.Cu") (net 19))
   (segment (start 123.444 142.528) (end 143.002 142.528) (width 0.3) (layer "F.Cu") (net 19))
   (segment (start 161.832 142.528) (end 162.052 142.528) (width 0.3) (layer "F.Cu") (net 19))
@@
   (segment (start 168.656 145.156) (end 168.915 145.415) (width 0.3) (layer "B.Cu") (net 30))
   (segment (start 177.292 132.588) (end 168.656 141.224) (width 0.3) (layer "B.Cu") (net 30))
-  (segment (start 171.455 140.203) (end 171.455 145.415) (width 0.3) (layer "F.Cu") (net 31))
+  (segment (start 171.455 137.155) (end 171.455 145.415) (width 0.3) (layer "F.Cu") (net 31))
+  (segment (start 180.086 112.776) (end 180.086 124.54296) (width 0.3) (layer "F.Cu") (net 31))
+  (segment (start 180.086 124.54296) (end 177.292 127.33696) (width 0.3) (layer "F.Cu") (net 31))
   (segment (start 161.925 103.48) (end 161.798 103.607) (width 0.3) (layer "F.Cu") (net 31))
-  (segment (start 180.086 112.776) (end 180.34 113.03) (width 0.3) (layer "F.Cu") (net 31))
-  (segment (start 180.34 113.03) (end 180.34 131.318) (width 0.3) (layer "F.Cu") (net 31))
   (segment (start 174.752 112.776) (end 178.054 112.776) (width 0.3) (layer "F.Cu") (net 31))
   (segment (start 161.798 103.607) (end 161.798 104.902) (width 0.3) (layer "F.Cu") (net 31))
-  (segment (start 180.34 131.318) (end 171.455 140.203) (width 0.3) (layer "F.Cu") (net 31))
+  (segment (start 177.292 127.33696) (end 177.292 131.318) (width 0.3) (layer "F.Cu") (net 31))
+  (segment (start 177.292 131.318) (end 171.455 137.155) (width 0.3) (layer "F.Cu") (net 31))
   (via (at 178.054 112.776) (size 0.8) (drill 0.4) (layers "F.Cu" "B.Cu") (net 31))
   (via (at 161.798 104.902) (size 0.8) (drill 0.4) (layers "F.Cu" "B.Cu") (net 31))
@@
   (segment (start 164.592 107.696) (end 169.672 107.696) (width 0.3) (layer "B.Cu") (net 31))
   (segment (start 178.054 112.776) (end 180.086 112.776) (width 0.3) (layer "B.Cu") (net 31))
-  (segment (start 173.995 139.441) (end 181.102 132.334) (width 0.3) (layer "F.Cu") (net 32))
-  (segment (start 181.102 89.662) (end 179.7 88.26) (width 0.3) (layer "F.Cu") (net 32))
+  (segment (start 180.835511 132.600489) (end 180.835511 89.395511) (width 0.3) (layer "F.Cu") (net 32))
+  (segment (start 173.995 139.441) (end 180.835511 132.600489) (width 0.3) (layer "F.Cu") (net 32))
+  (segment (start 180.835511 89.395511) (end 179.7 88.26) (width 0.3) (layer "F.Cu") (net 32))
+  (segment (start 179.7 88.26) (end 177.66 88.26) (width 0.3) (layer "F.Cu") (net 32))
   (segment (start 173.995 145.415) (end 173.995 139.441) (width 0.3) (layer "F.Cu") (net 32))
-  (segment (start 179.7 88.26) (end 177.66 88.26) (width 0.3) (layer "F.Cu") (net 32))
-  (segment (start 181.102 132.334) (end 181.102 89.662) (width 0.3) (layer "F.Cu") (net 32))
-  (segment (start 176.535 138.425) (end 181.864 133.096) (width 0.3) (layer "F.Cu") (net 33))
-  (segment (start 180.34 86.868) (end 177.782 86.868) (width 0.3) (layer "F.Cu") (net 33))
-  (segment (start 176.535 145.415) (end 176.535 138.425) (width 0.3) (layer "F.Cu") (net 33))
-  (segment (start 181.864 133.096) (end 181.864 88.392) (width 0.3) (layer "F.Cu") (net 33))
-  (segment (start 177.782 86.868) (end 177.66 86.99) (width 0.3) (layer "F.Cu") (net 33))
-  (segment (start 181.864 88.392) (end 180.34 86.868) (width 0.3) (layer "F.Cu") (net 33))
+  (segment (start 177.792 87.122) (end 177.66 86.99) (width 0.3) (layer "F.Cu") (net 33))
+  (segment (start 179.959 87.122) (end 177.792 87.122) (width 0.3) (layer "F.Cu") (net 33))
+  (via (at 179.959 87.122) (size 0.8) (drill 0.4) (layers "F.Cu" "B.Cu") (net 33))
+  (segment (start 180.835511 109.461511) (end 180.721 109.347) (width 0.3) (layer "B.Cu") (net 33))
+  (segment (start 180.721 109.347) (end 180.721 87.884) (width 0.3) (layer "B.Cu") (net 33))
+  (segment (start 180.721 87.884) (end 179.959 87.122) (width 0.3) (layer "B.Cu") (net 33))
+  (segment (start 180.835511 114.566489) (end 180.835511 109.461511) (width 0.3) (layer "B.Cu") (net 33))
+  (segment (start 180.467 141.483) (end 180.467 114.935) (width 0.3) (layer "B.Cu") (net 33))
+  (segment (start 176.535 145.415) (end 180.467 141.483) (width 0.3) (layer "B.Cu") (net 33))
+  (segment (start 180.467 114.935) (end 180.835511 114.566489) (width 0.3) (layer "B.Cu") (net 33))
   (segment (start 173.99 104.902) (end 176.472022 104.902) (width 0.3) (layer "F.Cu") (net 34))
   (segment (start 142.707 88.138) (end 140.589 86.02) (width 0.3) (layer "F.Cu") (net 34))
